File: hardware/pcb/domofon.kicad_pcb (KiCad board)
At the start: 2 copper layers, 55.5 x 45.9 mm, 31 parts, among them J1 MTJ-642BX2, K1 AQY212GH, T1 LM-NP-1001-B1L, U1 LTV-814, X1 XY308-2P LINIA, X2 XY308-2P 5V/GND

Commit message: Update DTMF transmit parts and firmware sources.
C2/C3 are 220 nF with R6 100 Ω and R8 330 Ω (C5 stays 1 µF) so the sine PWM at 200 kHz is louder and still filtered. Firmware uses esphome-dtmf-tone and esphome-dtmf-decoder instead of the vendored decoder.
Parts:
- C2, C3: value 47n -> 220n
- R6a, R6b: value 1k -> 100R
- R8a, R8b: value 2k2 -> 330R
Changed lines of the file:
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@@
 			)
 		)
-		(property "Value" "47n"
+		(property "Value" "220n"
 			(at 0 1.199999 0)
 			(layer "F.Fab")
@@
 			)
 		)
-		(property "Value" "2k2"
+		(property "Value" "330R"
 			(at 1.199999 0 0)
 			(layer "F.Fab")
@@
 			)
 		)
-		(property "Value" "1k"
+		(property "Value" "100R"
 			(at 1.2 0 0)
 			(layer "F.Fab")
@@
 			)
 		)
-		(property "Value" "1k"
+		(property "Value" "100R"
 			(at 1.199999 0 0)
 			(layer "F.Fab")
@@
 			)
 		)
-		(property "Value" "47n"
+		(property "Value" "220n"
 			(at -1.2 0 0)
 			(layer "F.Fab")
@@
 			)
 		)
-		(property "Value" "2k2"
+		(property "Value" "330R"
 			(at 1.2 0 0)
 			(layer "F.Fab")

Commit message: Consistency pass rev. 5: C8 replaces R2 on PCB (same pads), K1 AQY214EH, D2 P6KE220CA, C5 1u/100V in KiCad/generators/gerbers/enclosure; docs/BOM cleanup; schematic PNG ~3200 px
Parts:
- C5: value 1u/63V -> 1u/100V
- C8: renamed from R2; value 4k7 -> 470n/250V; footprint domofon:R0207_P7.62 -> domofon:CFILM_P7.62
- D2: value P6KE36CA -> P6KE220CA
- K1: value AQY212GH -> AQY214EH
Connections:
- net N_R12 renamed N_C8R1
Changed lines of the file:
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@@
 	(net 1 "L1")
 	(net 2 "L2")
-	(net 3 "N_R12")
+	(net 3 "N_C8R1")
 	(net 4 "N_U1A")
 	(net 5 "H")
@@
 		(embedded_fonts no)
 	)
-	(footprint "domofon:R0207_P7.62"
+	(footprint "domofon:CFILM_P7.62"
 		(layer "F.Cu")
 		(at 43 19.2)
-		(property "Reference" "R2"
+		(property "Reference" "C8"
 			(at 0 0 0)
 			(layer "F.SilkS")
@@
 			)
 		)
-		(property "Value" "4k7"
+		(property "Value" "470n/250V"
 			(at 0 1.2 0)
 			(layer "F.Fab")
@@
 			(layers "B.Cu" "B.Mask")
 			(remove_unused_layers no)
-			(net 3 "N_R12")
+			(net 3 "N_C8R1")
 		)
 		(embedded_fonts no)
@@
 			)
 		)
-		(property "Value" "1u/63V"
+		(property "Value" "1u/100V"
 			(at 0 1.2 0)
 			(layer "F.Fab")
@@
 			)
 		)
-		(property "Value" "AQY212GH"
+		(property "Value" "AQY214EH"
 			(at 0 1.2 0)
 			(layer "F.Fab")
@@
 			)
 		)
-		(property "Value" "P6KE36CA"
+		(property "Value" "P6KE220CA"
 			(at 0 1.2 0)
 			(layer "F.Fab")
@@
 			(layers "B.Cu" "B.Mask")
 			(remove_unused_layers no)
-			(net 3 "N_R12")
+			(net 3 "N_C8R1")
 		)
 		(pad "2" thru_hole circle
